Commit message: minor refactoring to make it easier to go where I need to go next

File: urdf/my_HAP.xacro (robot description, xacro)
@@ -14,5 +14,5 @@
       </inertial>
   </xacro:macro>
-  <xacro:macro name="Livox_HAP_gazebo_sensor" params="visualize:=True update_rate:=10 resolution:=0.002 noise_mean:=0.0 noise_stddev:=0.01 name:=livox">
+  <xacro:macro name="Livox_HAP_gazebo_sensor" params="name:=livox visualize:=True update_rate:=10 resolution:=0.002 noise_mean:=0.0 noise_stddev:=0.01">
     <gazebo reference="${name}">
       <sensor type="ray" name="${name}_lidar">
@@ -57,5 +57,5 @@
     </gazebo>
   </xacro:macro>
-  <xacro:macro name="Livox_HAP" params="visualize:=True name:=livox">
+  <xacro:macro name="Livox_HAP" params="name:=livox visualize:=True">
     <link name="${name}_base">
       <xacro:null_inertial/>
@@ -83,4 +83,4 @@
     <xacro:Livox_HAP_gazebo_sensor name="${name}" visualize="${visualize}"/>
   </xacro:macro>
-  <xacro:Livox_HAP name="livox"/>
+  <xacro:Livox_HAP name="livox" />
 </robot>

Commit message: adding laser_retro + custom laser reflections

File: urdf/my_HAP.xacro (robot description, xacro)
@@ -61,5 +61,5 @@
       <xacro:null_inertial/>
       <visual>
-        <origin xyz="-0.0445 0 0.032.5" rpy="0 ${pi/2} 0" />
+        <origin xyz="-0.0445 0 0.0325" rpy="0 ${pi/2} 0" />
         <geometry>
           <mesh filename="package://livox_laser_simulation/meshes/livox_HAP.dae" scale=".001 .001 .001" />
@@ -67,5 +67,5 @@
       </visual>
       <collision>
-		    <origin xyz="-0.0445 0 0.032.5" rpy="0 0 0" />
+		    <origin xyz="-0.0445 0 0.0325" rpy="0 0 0" />
         <geometry>
           <box size="0.105 0.1316 0.065"/>

Commit message: removed most of the unused code to make the module GOFAST

File: urdf/my_HAP.xacro (robot description, xacro)
@@ -14,5 +14,5 @@
       </inertial>
   </xacro:macro>
-  <xacro:macro name="Livox_HAP_gazebo_sensor" params="name:=livox visualize:=True update_rate:=10 resolution:=0.002 noise_mean:=0.0 noise_stddev:=0.01">
+  <xacro:macro name="Livox_HAP_gazebo_sensor" params="name:=livox visualize:=True update_rate:=10 resolution:=0.002 noise_mean:=0.0 noise_stddev:=0.005">
     <gazebo reference="${name}">
       <sensor type="ray" name="${name}_lidar">
@@ -20,42 +20,41 @@
         <visualize>${visualize}</visualize>
         <update_rate>${update_rate}</update_rate>
-        <!-- This ray plgin is only for visualization. -->
+        <ray>
+          <scan>
+            <horizontal>
+              <samples>${samples}</samples> <!-- tag is ignored by plugin -->
+              <resolution>1</resolution>
+              <min_angle>${-60/180*pi}</min_angle>
+              <max_angle>${60/180*pi}</max_angle>
+            </horizontal>
+            <vertical>
+              <samples>1</samples> <!-- tag is ignored by plugin -->
+              <resolution>1</resolution>
+              <min_angle>${-12.5/180*pi}</min_angle>
+              <max_angle>${12.5/180*pi}</max_angle>
+            </vertical>
+          </scan>
+          <range>
+            <min>${laser_min_range}</min>
+            <max>${laser_max_range}</max>
+            <resolution>${resolution}</resolution>
+          </range>
+          <noise>
+            <type>gaussian</type>
+            <mean>${noise_mean}</mean>
+            <stddev>${noise_stddev}</stddev>
+          </noise>
+        </ray>
         <plugin name="gazebo_ros_laser_controller" filename="liblivox_laser_simulation.so">
-          <ray>
-            <scan>
-              <horizontal>
-                <samples>100</samples>
-                <resolution>1</resolution>
-                <min_angle>${-60/180*pi}</min_angle>
-                <max_angle>${60/180*pi}</max_angle>
-              </horizontal>
-              <vertical>
-                <samples>50</samples>
-                <resolution>1</resolution>
-                <min_angle>${-12.5/180*pi}</min_angle>
-                <max_angle>${12.5/180*pi}</max_angle>
-              </vertical>
-            </scan>
-            <range>
-              <min>${laser_min_range}</min>
-              <max>${laser_max_range}</max>
-              <resolution>${resolution}</resolution>
-            </range>
-            <noise>
-              <type>gaussian</type>
-              <mean>${noise_mean}</mean>
-              <stddev>${noise_stddev}</stddev>
-            </noise>
-          </ray>
-          <visualize>${visualize}</visualize>
+          <topicName>/${name}/lidar</topicName>
+          <!-- <frameName>${name}_sensor</frameName> -->
+          <frameName>lidar</frameName>
           <samples>${samples}</samples>
-          <downsample>${downsample}</downsample>
           <csv_file_name>package://livox_laser_simulation/scan_mode/HAP.csv</csv_file_name>
-          <ros_topic>${ros_topic}</ros_topic>
         </plugin>
       </sensor>
     </gazebo>
   </xacro:macro>
-  <xacro:macro name="Livox_HAP" params="name:=livox visualize:=True">
+  <xacro:macro name="Livox_HAP" params="name:=livox visualize:=False">
     <link name="${name}_base">
       <xacro:null_inertial/>
@@ -83,4 +82,5 @@
     <xacro:Livox_HAP_gazebo_sensor name="${name}" visualize="${visualize}"/>
   </xacro:macro>
+  <!--Note : default visualize=false is recommended, as the visualization is a bit wonky-->
   <xacro:Livox_HAP name="livox" />
 </robot>

Commit message: formatting XML

File: urdf/my_HAP.xacro (robot description, xacro)
@@ -1,18 +1,19 @@
 <?xml version="1.0"?>
 <robot xmlns:xacro="http://ros.org/wiki/xacro">
-  <xacro:property name="laser_min_range" value="0.1"/>
-  <xacro:property name="laser_max_range" value="200.0"/>
-  <xacro:property name="ros_topic" value="livox/lidar"/>
+  <xacro:property name="laser_min_range" value="0.1" />
+  <xacro:property name="laser_max_range" value="200.0" />
+  <xacro:property name="ros_topic" value="livox/lidar" />
   <xacro:property name="samples" value="45300"/>
-  <xacro:property name="downsample" value="1"/>
+  <xacro:property name="downsample" value="1" />
   <xacro:macro name="null_inertial">
     <inertial>
-      <mass value="0.1"/>
+      <mass value="0.1" />
       <inertia ixx="0.01" ixy="0" ixz="0"
-            iyy="0.01" iyz="0"
-            izz="0.01"/>
-      </inertial>
+        iyy="0.01" iyz="0"
+        izz="0.01" />
+    </inertial>
   </xacro:macro>
-  <xacro:macro name="Livox_HAP_gazebo_sensor" params="name:=livox visualize:=True update_rate:=10 resolution:=0.002 noise_mean:=0.0 noise_stddev:=0.01">
+  <xacro:macro name="Livox_HAP_gazebo_sensor"
+    params="name:=livox visualize:=True update_rate:=10 resolution:=0.002 noise_mean:=0.0 noise_stddev:=0.01">
     <gazebo reference="${name}">
       <sensor type="ray" name="${name}_lidar">
@@ -59,27 +60,30 @@
   <xacro:macro name="Livox_HAP" params="name:=livox visualize:=True">
     <link name="${name}_base">
-      <xacro:null_inertial/>
+      <xacro:null_inertial />
       <visual>
         <origin xyz="-0.0445 0 0.0325" rpy="0 ${pi/2} 0" />
         <geometry>
-          <mesh filename="package://livox_laser_simulation/meshes/livox_HAP.dae" scale=".001 .001 .001" />
+          <mesh
+            filename="package://livox_laser_simulation/meshes/livox_HAP.dae"
+            scale=".001 .001 .001"
+          />
         </geometry>
       </visual>
       <collision>
-		    <origin xyz="-0.0445 0 0.0325" rpy="0 0 0" />
+        <origin xyz="-0.0445 0 0.0325" rpy="0 0 0" />
         <geometry>
-          <box size="0.105 0.1316 0.065"/>
+          <box size="0.105 0.1316 0.065" />
         </geometry>
       </collision>
     </link>
     <link name="${name}">
-      <xacro:null_inertial/>
+      <xacro:null_inertial />
     </link>
     <joint name="${name}_to_${name}_base_joint" type="fixed">
-      <parent link="${name}_base"/>
-      <child link="${name}"/>
-      <origin xyz="0.008 0 0.023" rpy="0 0 0"/>
+      <parent link="${name}_base" />
+      <child link="${name}" />
+      <origin xyz="0.008 0 0.023" rpy="0 0 0" />
     </joint>
-    <xacro:Livox_HAP_gazebo_sensor name="${name}" visualize="${visualize}"/>
+    <xacro:Livox_HAP_gazebo_sensor name="${name}" visualize="${visualize}" />
   </xacro:macro>
   <xacro:Livox_HAP name="livox" />
